File: 2key-keypad.kicad_pcb (KiCad board)
At the start: 2 copper layers, 38.1 x 46.8 mm, 20 parts, among them SW1 SW_Push, U1 ATmega32U4-A, Y1 16MHz

Commit message: Finished First Schem
Parts:
- MX1, MX2: footprint MX_Alps_Hybrid:MX-1U -> MX_Only:MXOnly-1U-Hotswap
Routing:
- net ROW0: track 0.00 -> 48.9 mm
- net COL0: track 0.00 -> 48.4 mm
- net COL1: track 0.00 -> 31.0 mm
- net GND: track 133.2 -> 106.8 mm
- net Net-(D2-A): track 0.00 -> 4.30 mm
- net Net-(D1-A): track 0.00 -> 4.30 mm
- added copper zone on B.Cu, net GND
