File: 2key-keypad2.0/2key-keypad2.0.kicad_sch (KiCad schematic)
At the start: 21 parts, among them SW1 SW_Push, U2 ATmega32U2-AU, Y1 16MHz

Commit message: V2.0
Parts:
- F1: value Polyfuse_Small -> 500mah
- SW1: footprint random-keyboard-parts:SOT143B -> random-keyboard-parts:SKQGADE010
Changed lines of the file:
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@@
       (effects (font (size 1.27 1.27)))
     )
-    (property "Footprint" "random-keyboard-parts:SOT143B" (at 36.83 31.75 0)
+    (property "Footprint" "random-keyboard-parts:SKQGADE010" (at 36.83 31.75 0)
       (effects (font (size 1.27 1.27)) hide)
     )
@@
       (effects (font (size 1.27 1.27)))
     )
-    (property "Value" "Polyfuse_Small" (at 138.43 81.28 90)
-      (effects (font (size 1.27 1.27)))
-    )
+    (property "Value" "500mah" (at 138.43 81.28 90)
+      (effects (font (size 1.27 1.27)))
+    )
